File: pulse.sch (EAGLE design)
At the start: 26 parts, among them IC1 AD8607R, IC2 AD8607R, Q1 DMN2215UDM-7, Q2 DMP2240UDM-7, Q3 BC817-16LT1G

Commit message: GND fixed
Connections:
- net GND: now also IC2P.V-
Changed lines of the file:
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@@
 <part name="R13" library="adafruit" deviceset="R-US_" device="M0805"/>
 <part name="GND6" library="supply1" deviceset="GND" device=""/>
+<part name="GND7" library="supply1" deviceset="GND" device=""/>
 </parts>
 <sheets>
@@
 <instance part="GND2" gate="1" x="91.44" y="63.5"/>
 <instance part="GND3" gate="1" x="12.7" y="76.2"/>
+<instance part="GND7" gate="1" x="40.64" y="71.12"/>
 </instances>
 <busses>
@@
 <wire x1="91.44" y1="66.04" x2="91.44" y2="71.12" width="0.1524" layer="91"/>
 </segment>
-</net>
+<segment>
+<pinref part="IC2" gate="P" pin="V-"/>
+<pinref part="GND7" gate="1" pin="GND"/>
+<wire x1="48.26" y1="73.66" x2="40.64" y2="73.66" width="0.1524" layer="91"/>
+</segment>
+</net>
